Commit message: Complete project structure reorganization and cleanup
Major improvements:
- Moved legacy code to legacy/ directory preserving historical examples
- Cleaned examples/ to focus on modern SimulationManager architecture
- Deleted redundant and conflicting files while maintaining functionality
- Updated all documentation to reflect new organization
- Added comprehensive CLAUDE.md for project memory

Architecture enhancements:
- Enhanced core/ modules with proper URDF visual origin processing
- Improved robot models with realistic 4-DOF arm structure
- Simplified user interface reducing code from ~100 lines to ~20 lines
- 89+ Hz performance with multi-robot support

File organization:
- examples/simple/ - Modern SimulationManager examples
- examples/robots/ - Enhanced URDF robot models
- legacy/ - Preserved historical code for reference
- core/ - Enhanced simulation architecture

🤖 Generated with [Claude Code](https://claude.ai/code)

Co-Authored-By: Claude <noreply@anthropic.com>

File: examples/robots/collision_robot.urdf (robot description, URDF)
Before this commit: robot simple_robot, 3 links, 2 joints
Joints:
- joint arm_to_end: origin xyz=0 0 0.35 rpy=0 0 0 -> xyz=0 0 0.6 rpy=0 0 0
- joint base_to_arm: axis 0 0 1 -> 0 1 0; origin xyz=0.2 0 0.1 rpy=0 0 0 -> xyz=0.25 0 0.10 rpy=0 0 0
